File: ParentBoard/ParentBoard.kicad_pcb (KiCad board)
At the start: 4 copper layers, 306 parts, among them J1 ShuntA, J10 Connector_A, J11 Connector_B, J12 Connector_C, J13 AH, J16 AH, J17 AH, J18 AH, J19 AH, J2 ShuntA, J20 AH, J21 AH, J22 AH, J23 AH, J24 AH, J25 AH, J26 AH, J27 Connector_B, J3 ShuntA, J4 AH, J5 AH, J6 AH, J7 AH, J8 AH, J9 AH, Q6 AOD413A, Q7 AOD413A, U1 OPA365xxDBV, U10 TL341, U11 AMC1301, U12 OPA365xxDBV, U13 AMC1311, U14 AMC1311, U15 AMC1311, U16 74LVC1G66, U17 74LVC1G66, U18 74LVC1G66, U19 74LVC1G66, U2 OPA365xxDBV, U20 74LVC1G66, U21 74LVC1G66, U22 74LVC1G66, U23 UCC21520DW, U24 UCC21520DW, U25 UCC21520DW, U26 AMC1311, U27 TL072, U28 TLC372, U29 TLC372, U3 OPA365xxDBV, U30 TLC372, U31 AMC1311, U32 AZ1117-5.0, U33 1769405241-2W-1205, U34 TLC372, U35 74AHC1G02, U36 74LVC1G11, U37 TL341, U38 TL341, U39 TL341, U4 AMC1301, U5 TL341, U6 OPA365xxDBV, U7 TL341, U8 AMC1301, U9 OPA365xxDBV

Commit message: routing pinheader
Parts:
- added J14: Conn_02x21_Odd_Even, Connector_PinHeader_2.54mm:PinHeader_2x21_P2.54mm_Vertical, F.Cu at (119.6, 52.3)
- added R65: 120, Resistor_SMD:R_0805_2012Metric_Pad1.20x1.40mm_HandSolder, F.Cu at (129.8, 38.0)
- added R66: 10k, Resistor_SMD:R_0805_2012Metric, F.Cu at (139.4, 43.9)
- added R67: 10k, Resistor_SMD:R_0805_2012Metric, F.Cu at (136.6, 43.6)
- added R68: 220, Resistor_SMD:R_0805_2012Metric_Pad1.20x1.40mm_HandSolder, F.Cu at (133.8, 44.2)
- added U40: MCP2562-E-SN, Package_SO:SOIC-8_3.9x4.9mm_P1.27mm, F.Cu at (129.9, 43.0)
- added U41: TL341, Package_TO_SOT_SMD:SOT-23-3, F.Cu at (134.6, 40.0)
- moved C84 334.9 mm to (239.3, 73.5), turned to 90 degrees
- moved C46 329.1 mm to (221.2, 70.4), turned to 90 degrees
- moved R44 316.1 mm to (218.4, 64.8), turned to -90 degrees
- moved R45 314.1 mm to (216.2, 64.8), turned to 90 degrees
- moved R46 309.9 mm to (212.1, 67.8), turned to 90 degrees
- moved R47 307.2 mm to (209.2, 66.6), turned to 180 degrees
- moved C47 283.2 mm to (223.7, 68.7), turned to 90 degrees
- moved C106 276.9 mm to (231.8, 55.6), turned to 180 degrees
- moved C105 274.9 mm to (229.8, 53.3), turned to 180 degrees
- moved C79 269.0 mm to (218.4, 69.0), turned to -90 degrees
- moved C72 267.5 mm to (165.3, 73.7), turned to 90 degrees
- moved C37 267.1 mm to (202.7, 64.0), turned to 90 degrees
- moved C80 266.7 mm to (216.2, 69.0), turned to 90 degrees
- moved C36 264.5 mm to (200.2, 61.8), turned to 90 degrees
- moved C82 259.4 mm to (209.1, 68.6), turned to 180 degrees
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Connections:
- R117 pad 2: /T+ -> /V+
- R118 pad 2: /T- -> /V-
- TP38 pad 1: /T+ -> /V+
- TP39 pad 1: /T- -> /V-
- U31 pad 6: /T- -> /V-
- U31 pad 7: /T+ -> /V+
Routing:
- net /D-: track 0.00 -> 81.3 mm
- net /D+: track 0.00 -> 77.3 mm
- net /CC-: track 0.00 -> 74.0 mm
- net /T+: track 0.00 -> 71.3 mm
- net /T-: track 0.00 -> 71.3 mm
- net /CC+: track 0.00 -> 71.2 mm
- net /CA+: track 0.00 -> 70.2 mm
- net /InAH: track 0.00 -> 68.3 mm
- net /D3-: track 0.00 -> 66.9 mm
- net /CA-: track 0.00 -> 66.9 mm
- net /InAL: track 0.00 -> 65.3 mm
- net /InCH: track 0.00 -> 64.7 mm
- net /V-: track 0.00 -> 63.2 mm
- net /V+: track 0.00 -> 63.1 mm
- net /D3+: track 0.00 -> 63.0 mm
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