File: ParentBoard/ParentBoard.kicad_sch (KiCad schematic)
At the start: 306 parts, among them J1 ShuntA, J10 Connector_A, J11 Connector_B, J12 Connector_C, J13 AH, J16 AH, J17 AH, J18 AH, J19 AH, J2 ShuntA, J20 AH, J21 AH, J22 AH, J23 AH, J24 AH, J25 AH, J26 AH, J27 Connector_B, J3 ShuntA, J4 AH, J5 AH, J6 AH, J7 AH, J8 AH, J9 AH, Q6 AOD413A, Q7 AOD413A, U1 OPA365xxDBV, U10 TL341, U11 AMC1301, U12 OPA365xxDBV, U13 AMC1311, U14 AMC1311, U15 AMC1311, U16 74LVC1G66, U17 74LVC1G66, U18 74LVC1G66, U19 74LVC1G66, U2 OPA365xxDBV, U20 74LVC1G66, U21 74LVC1G66, U22 74LVC1G66, U23 UCC21520DW, U24 UCC21520DW, U25 UCC21520DW, U26 AMC1311, U27 TL072, U28 TLC372, U29 TLC372, U3 OPA365xxDBV, U30 TLC372, U31 AMC1311, U32 AZ1117-5.0, U33 1769405241-2W-1205, U34 TLC372, U35 74AHC1G02, U36 74LVC1G11, U37 TL341, U38 TL341, U39 TL341, U4 AMC1301, U5 TL341, U6 OPA365xxDBV, U7 TL341, U8 AMC1301, U9 OPA365xxDBV

Commit message: routing pinheader
Parts:
- added C109, C110: 100nF, symbol Device:C_Small
- added J14: Conn_02x21_Odd_Even, Connector_PinHeader_2.54mm:PinHeader_2x21_P2.54mm_Vertical, symbol Connector_Generic:Conn_02x21_Odd_Even
- added R65: 120, Resistor_SMD:R_0805_2012Metric_Pad1.20x1.40mm_HandSolder, symbol Device:R
- added R66, R67: 10k, Resistor_SMD:R_0805_2012Metric, symbol Device:R
- added R68: 220, Resistor_SMD:R_0805_2012Metric_Pad1.20x1.40mm_HandSolder, symbol Device:R
- added U40: MCP2562-E-SN, Package_SO:SOIC-8_3.9x4.9mm_P1.27mm, symbol Interface_CAN_LIN:MCP2562-E-SN
- added U41: TL341, Package_TO_SOT_SMD:SOT-23-3, symbol Reference_Voltage:LM285M-ADJ
Connections:
- net +5V: now also C110.2, J14.19 (Pin_19), J14.20 (Pin_20), J14.21 (Pin_21), J14.22 (Pin_22), J14.23 (Pin_23), J14.24 (Pin_24), R68.1, U40.3 (VDD)
- net CA+: now also J14.12 (Pin_12)
- net CA-: now also J14.11 (Pin_11)
- net CB+: now also J14.30 (Pin_30)
- net CB-: now also J14.29 (Pin_29)
- net CC+: now also J14.39 (Pin_39)
- net CC-: now also J14.40 (Pin_40)
- net D+: now also J14.3 (Pin_3)
- net D-: now also J14.4 (Pin_4)
- net D2+: now also J14.13 (Pin_13)
- net D2-: now also J14.14 (Pin_14)
- net D3+: now also J14.31 (Pin_31)
- net D3-: now also J14.32 (Pin_32)
- net GND: now also C109.1, C110.1, J14.10 (Pin_10), J14.15 (Pin_15), J14.16 (Pin_16), J14.27 (Pin_27), J14.28 (Pin_28), J14.33 (Pin_33), J14.34 (Pin_34), J14.37 (Pin_37), J14.38 (Pin_38), J14.5 (Pin_5), J14.6 (Pin_6), J14.9 (Pin_9), R66.1, U40.2 (VSS), U40.8 (STBY), U41.3 (A)
- net InAH: now also J14.8 (Pin_8)
- net InAL: now also J14.7 (Pin_7)
- net InBH: now also J14.25 (Pin_25)
- net InBL: now also J14.26 (Pin_26)
- net InCH: now also J14.36 (Pin_36)
- net InCL: now also J14.35 (Pin_35)
- net T+: now also J14.2 (Pin_2); no longer R117.2, TP38.1, U31.7
- net T-: now also J14.1 (Pin_1); no longer R118.2, TP39.1, U31.6
- new net: R66.2, R67.1, U41.2 (REF)
- new net +3.3V: C109.2, R67.2, R68.2, U40.5 (Vio), U41.1 (K)
- new net CANH+: R65.1, U40.7 (CANH)
- new net CANL-: R65.2, U40.6 (CANL)
- new net CANRX: J14.17 (Pin_17), U40.4 (RXD)
- new net CANTX: J14.18 (Pin_18), U40.1 (TXD)
- new net V+: J14.41 (Pin_41), R117.2, TP38.1, U31.7
- new net V-: J14.42 (Pin_42), R118.2, TP39.1, U31.6
