File: PowerStage/PowerStage.kicad_pcb (KiCad board)
At the start: 2 copper layers, 87 parts, among them J1 AH, J10 AH, J11 AH, J12 AH, J13 AH, J14 AH, J19 PhaseA, J2 AH, J20 PhaseB, J21 PhaseB, J22 AH, J23 AH, J24 AH, J25 AH, J3 BH, J4 BH, J5 BH, J6 CH, J7 CH, J8 CH, J9 AH, Q20 HY5110W, Q21 HY5110W, Q22 HY5110W, Q23 HY5110W, Q24 HY5110W, Q25 HY5110W, Q26 HY5110W, Q27 HY5110W, Q28 HY5110W, Q29 HY5110W, Q30 HY5110W, Q31 HY5110W, Q38 HY5110W, Q39 HY5110W, Q40 HY5110W, Q41 HY5110W, Q42 HY5110W, Q43 HY5110W

Commit message: routing pinheader
Parts:
- added J15: CurrentA, Connector_PinSocket_2.54mm:PinSocket_1x02_P2.54mm_Vertical_SMD_Pin1Left, F.Cu at (83.3, 136.8)
- added J16: CurrentB, Connector_PinSocket_2.54mm:PinSocket_1x02_P2.54mm_Vertical_SMD_Pin1Left, F.Cu at (157.4, 136.6)
- added J17: CurrentC, Connector_PinSocket_2.54mm:PinSocket_1x02_P2.54mm_Vertical_SMD_Pin1Left, F.Cu at (231.4, 136.2)
- added J18: Terminal A, custom:225685-E, F.Cu at (57.1, 155.4)
- added J26: Terminal B, custom:225685-E, F.Cu at (131.3, 155.5)
- added J27: Terminal C, custom:225685-E, F.Cu at (205.2, 155.5)
- added R17: 1m, custom:ShuntResistor_P2mmD10mm, F.Cu at (62.0, 140.6)
- added R19: 1m, custom:ShuntResistor_P2mmD10mm, F.Cu at (57.0, 140.6)
- added R28: 1m, custom:ShuntResistor_P2mmD10mm, F.Cu at (52.0, 140.6)
- added R29: 1m, custom:ShuntResistor_P2mmD10mm, F.Cu at (136.2, 140.6)
- added R30: 1m, custom:ShuntResistor_P2mmD10mm, F.Cu at (131.2, 140.6)
- added R31: 1m, custom:ShuntResistor_P2mmD10mm, F.Cu at (126.2, 140.6)
- added R32: 1m, custom:ShuntResistor_P2mmD10mm, F.Cu at (210.2, 140.6)
- added R33: 1m, custom:ShuntResistor_P2mmD10mm, F.Cu at (205.2, 140.6)
- added R34: 1m, custom:ShuntResistor_P2mmD10mm, F.Cu at (200.2, 140.6)
- C14, C15, C16, C17: value 820u_100v -> 470u_200v; footprint Capacitor_THT:CP_Radial_D18.0mm_P7.50mm -> Capacitor_THT:CP_Radial_D25.0mm_P10.00mm_SnapIn
- J19: value PhaseA -> phaseA+
- J20, J21: value PhaseB -> phaseB+
- moved C16 75.2 mm to (239.0, 50.2)
- moved C14 65.6 mm to (193.4, 49.3)
- moved C15 36.5 mm to (41.9, 41.9)
- moved C17 31.8 mm to (78.6, 40.2)
- moved R4 24.4 mm to (30.8, 91.2)
- moved R21 20.6 mm to (31.0, 113.7)
Connections:
- net /phaseA renamed /phaseA+
- net /phaseB renamed /phaseB+
- net /phaseC renamed /phaseC+
Routing:
- net /phaseA+: track 11.1 -> 24.2 mm
- net /phaseC+: track 11.1 -> 24.2 mm
- net /phaseB+: track 11.2 -> 23.2 mm
- net /CL1: track 0.00 -> 6.01 mm
- net /AL2: track 0.00 -> 6.00 mm
- net /AL1: track 0.00 -> 5.92 mm
- net /CL2: track 0.00 -> 5.81 mm
- net /BH1: track 0.00 -> 3.96 mm
- net /CH1: track 0.00 -> 3.89 mm
- net /AH2: track 0.00 -> 3.88 mm
- net /CH2: track 0.00 -> 3.84 mm
- net /BH3: track 0.00 -> 3.80 mm
- net /BH2: track 0.00 -> 3.80 mm
- net /AH3: track 0.00 -> 3.71 mm
- net /CH3: track 0.00 -> 3.65 mm
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- added copper zone on F.Cu, net /AH1
- added copper zone on F.Cu, net /AH2
- added copper zone on F.Cu, net /AH3
- added copper zone on F.Cu, net /AL1
- added copper zone on F.Cu, net /AL2
- added copper zone on F.Cu, net /AL3
- added copper zone on F.Cu, net /BH1
- added copper zone on F.Cu, net /BH2
- added copper zone on F.Cu, net /BH3
- added copper zone on F.Cu, net /BL1
- added copper zone on F.Cu, net /BL2
- added copper zone on F.Cu, net /BL3
- added copper zone on F.Cu, net /CH1
- added copper zone on F.Cu, net /CH2
- added copper zone on F.Cu, net /CH3
- added copper zone on F.Cu, net /CL1
- added copper zone on F.Cu, net /CL2
- added copper zone on F.Cu, net /CL3
- added copper zone on F.Cu, net /phaseA+
- added copper zone on B.Cu, net /phaseA-
- added copper zone on F.Cu, net /phaseA-
- added copper zone on F.Cu, net /phaseB+
- added copper zone on B.Cu, net /phaseB-
- added copper zone on F.Cu, net /phaseB-
- added copper zone on F.Cu, net /phaseC+
- added copper zone on B.Cu, net /phaseC-
- added copper zone on F.Cu, net /phaseC-
- added copper zone on B.Cu, net GND
- added copper zone on F.Cu, net GND
- added copper zone on B.Cu, net V+
Other:
- board text added: "J2"
